Commit message: fine tune offset test and fix constant velocity test

File: source/extensions/omni.isaac.lab/test/sensors/urdfs/simple_2_link.urdf (robot description, URDF)
Before this commit: robot simple_2_link, 4 links, 3 joints
Links:
- link base: geometry visual cylinder length=0.6 radius=0.015
- link imu_link: mass 0.001 -> 0.00001
- link link_1: geometry visual cylinder length=0.4 radius=0.01
Joints:
- joint imu_joint: origin xyz=0.4 0.0 0.25 rpy=1.57079632679 0 1.57087963 -> xyz=0.4 0.0 0.1 rpy=1.57079632679 0 1.57087963
